File: Adapter-RJ45-SignalHead.brd (EAGLE design)
At the start: 33 x 45.7 mm, 12 parts

Commit message: added values for connectors
Parts:
- CON1, CON2: value (none) -> 2mm
- CON3, CON4: value (none) -> 0.100
- J1: value (none) -> RJ12/6
- R1, R2, R3, R4, R5, R6: value (none) -> 0R
Changed lines of the file:
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@@
 <elements>
 <element name="U$1" library="SPCoast" package="OSHW-LOGO-M" value="DOC-OSHW-LOGO-M" x="16.51" y="41.91"/>
-<element name="CON1" library="SPCoast" package="4P-2.0" value="" x="26.035" y="9.525" smashed="yes">
+<element name="CON1" library="SPCoast" package="4P-2.0" value="2mm" x="26.035" y="9.525" smashed="yes">
 <attribute name="NAME" x="24.13" y="12.065" size="0.8128" layer="25" font="vector" ratio="11"/>
 </element>
-<element name="CON2" library="SPCoast" package="4P-2.0" value="" x="6.35" y="9.525" smashed="yes">
+<element name="CON2" library="SPCoast" package="4P-2.0" value="2mm" x="6.35" y="9.525" smashed="yes">
 <attribute name="NAME" x="4.445" y="12.065" size="0.889" layer="25" font="vector" ratio="11"/>
 </element>
-<element name="R1" library="SPCoast" package="CUT-R" value="" x="11.43" y="20.32" smashed="yes" rot="R90">
+<element name="R1" library="SPCoast" package="CUT-R" value="0R" x="11.43" y="20.32" smashed="yes" rot="R90">
 <attribute name="VALUE" x="10.16" y="20.32" size="0.4064" layer="27" font="vector" rot="R90"/>
 <attribute name="NAME" x="10.16" y="16.51" size="0.4064" layer="25" font="vector" rot="R90"/>
 </element>
-<element name="R2" library="SPCoast" package="CUT-R" value="" x="7.62" y="20.32" smashed="yes" rot="R90">
+<element name="R2" library="SPCoast" package="CUT-R" value="0R" x="7.62" y="20.32" smashed="yes" rot="R90">
 <attribute name="VALUE" x="6.35" y="20.32" size="0.4064" layer="27" font="vector" rot="R90"/>
 <attribute name="NAME" x="6.35" y="16.51" size="0.4064" layer="25" font="vector" rot="R90"/>
 </element>
-<element name="R3" library="SPCoast" package="CUT-R" value="" x="3.81" y="20.32" smashed="yes" rot="R90">
+<element name="R3" library="SPCoast" package="CUT-R" value="0R" x="3.81" y="20.32" smashed="yes" rot="R90">
 <attribute name="VALUE" x="2.54" y="20.32" size="0.4064" layer="27" font="vector" rot="R90"/>
 <attribute name="NAME" x="2.54" y="16.51" size="0.4064" layer="25" font="vector" rot="R90"/>
 </element>
-<element name="R4" library="SPCoast" package="CUT-R" value="" x="26.67" y="20.32" smashed="yes" rot="R90">
+<element name="R4" library="SPCoast" package="CUT-R" value="0R" x="26.67" y="20.32" smashed="yes" rot="R90">
 <attribute name="VALUE" x="25.4" y="20.32" size="0.4064" layer="27" font="vector" rot="R90"/>
 <attribute name="NAME" x="25.4" y="16.51" size="0.4064" layer="25" font="vector" rot="R90"/>
 </element>
-<element name="R5" library="SPCoast" package="CUT-R" value="" x="22.86" y="20.32" smashed="yes" rot="R90">
+<element name="R5" library="SPCoast" package="CUT-R" value="0R" x="22.86" y="20.32" smashed="yes" rot="R90">
 <attribute name="VALUE" x="21.59" y="20.32" size="0.4064" layer="27" font="vector" rot="R90"/>
 <attribute name="NAME" x="21.59" y="16.51" size="0.4064" layer="25" font="vector" rot="R90"/>
 </element>
-<element name="R6" library="SPCoast" package="CUT-R" value="" x="19.05" y="20.32" smashed="yes" rot="R90">
+<element name="R6" library="SPCoast" package="CUT-R" value="0R" x="19.05" y="20.32" smashed="yes" rot="R90">
 <attribute name="VALUE" x="17.78" y="20.32" size="0.4064" layer="27" font="vector" rot="R90"/>
 <attribute name="NAME" x="17.78" y="16.51" size="0.4064" layer="25" font="vector" rot="R90"/>
 </element>
-<element name="J1" library="SPCoast" package="RJ45-NO-SHIELD" value="" x="16.51" y="40.005" rot="R180">
+<element name="J1" library="SPCoast" package="RJ45-NO-SHIELD" value="RJ12/6" x="16.51" y="40.005" rot="R180">
 <attribute name="OPL" value="none" x="16.51" y="40.005" size="1.778" layer="27" font="vector" ratio="10" rot="R180" display="off"/>
 <attribute name="AMP" value="520151-4" x="16.51" y="40.005" size="1.778" layer="27" font="vector" ratio="10" rot="R180" display="off"/>
 </element>
-<element name="CON3" library="SPCoast" package="1X04_LOCK" value="" x="2.54" y="6.985"/>
-<element name="CON4" library="SPCoast" package="1X04_LOCK" value="" x="21.59" y="6.985"/>
+<element name="CON3" library="SPCoast" package="1X04_LOCK" value="0.100" x="2.54" y="6.985"/>
+<element name="CON4" library="SPCoast" package="1X04_LOCK" value="0.100" x="21.59" y="6.985"/>
 </elements>
 <signals>

Commit message: normalized values
Parts:
- J1: value RJ12/6 -> RJ45
- R1, R2, R3, R4, R5, R6: value 0R -> nostuff
- U$1: value DOC-OSHW-LOGO-M -> OSHW
Changed lines of the file:
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@@
 </autorouter>
 <elements>
-<element name="U$1" library="SPCoast" package="OSHW-LOGO-M" value="DOC-OSHW-LOGO-M" x="16.51" y="41.91"/>
+<element name="U$1" library="SPCoast" package="OSHW-LOGO-M" value="OSHW" x="16.51" y="41.91"/>
 <element name="CON1" library="SPCoast" package="4P-2.0" value="2mm" x="26.035" y="9.525" smashed="yes">
 <attribute name="NAME" x="24.13" y="12.065" size="0.8128" layer="25" font="vector" ratio="11"/>
@@
 <attribute name="NAME" x="4.445" y="12.065" size="0.889" layer="25" font="vector" ratio="11"/>
 </element>
-<element name="R1" library="SPCoast" package="CUT-R" value="0R" x="11.43" y="20.32" smashed="yes" rot="R90">
+<element name="R1" library="SPCoast" package="CUT-R" value="nostuff" x="11.43" y="20.32" smashed="yes" rot="R90">
 <attribute name="VALUE" x="10.16" y="20.32" size="0.4064" layer="27" font="vector" rot="R90"/>
 <attribute name="NAME" x="10.16" y="16.51" size="0.4064" layer="25" font="vector" rot="R90"/>
 </element>
-<element name="R2" library="SPCoast" package="CUT-R" value="0R" x="7.62" y="20.32" smashed="yes" rot="R90">
+<element name="R2" library="SPCoast" package="CUT-R" value="nostuff" x="7.62" y="20.32" smashed="yes" rot="R90">
 <attribute name="VALUE" x="6.35" y="20.32" size="0.4064" layer="27" font="vector" rot="R90"/>
 <attribute name="NAME" x="6.35" y="16.51" size="0.4064" layer="25" font="vector" rot="R90"/>
 </element>
-<element name="R3" library="SPCoast" package="CUT-R" value="0R" x="3.81" y="20.32" smashed="yes" rot="R90">
+<element name="R3" library="SPCoast" package="CUT-R" value="nostuff" x="3.81" y="20.32" smashed="yes" rot="R90">
 <attribute name="VALUE" x="2.54" y="20.32" size="0.4064" layer="27" font="vector" rot="R90"/>
 <attribute name="NAME" x="2.54" y="16.51" size="0.4064" layer="25" font="vector" rot="R90"/>
 </element>
-<element name="R4" library="SPCoast" package="CUT-R" value="0R" x="26.67" y="20.32" smashed="yes" rot="R90">
+<element name="R4" library="SPCoast" package="CUT-R" value="nostuff" x="26.67" y="20.32" smashed="yes" rot="R90">
 <attribute name="VALUE" x="25.4" y="20.32" size="0.4064" layer="27" font="vector" rot="R90"/>
 <attribute name="NAME" x="25.4" y="16.51" size="0.4064" layer="25" font="vector" rot="R90"/>
 </element>
-<element name="R5" library="SPCoast" package="CUT-R" value="0R" x="22.86" y="20.32" smashed="yes" rot="R90">
+<element name="R5" library="SPCoast" package="CUT-R" value="nostuff" x="22.86" y="20.32" smashed="yes" rot="R90">
 <attribute name="VALUE" x="21.59" y="20.32" size="0.4064" layer="27" font="vector" rot="R90"/>
 <attribute name="NAME" x="21.59" y="16.51" size="0.4064" layer="25" font="vector" rot="R90"/>
 </element>
-<element name="R6" library="SPCoast" package="CUT-R" value="0R" x="19.05" y="20.32" smashed="yes" rot="R90">
+<element name="R6" library="SPCoast" package="CUT-R" value="nostuff" x="19.05" y="20.32" smashed="yes" rot="R90">
 <attribute name="VALUE" x="17.78" y="20.32" size="0.4064" layer="27" font="vector" rot="R90"/>
 <attribute name="NAME" x="17.78" y="16.51" size="0.4064" layer="25" font="vector" rot="R90"/>
 </element>
-<element name="J1" library="SPCoast" package="RJ45-NO-SHIELD" value="RJ12/6" x="16.51" y="40.005" rot="R180">
+<element name="J1" library="SPCoast" package="RJ45-NO-SHIELD" value="RJ45" x="16.51" y="40.005" rot="R180">
 <attribute name="OPL" value="none" x="16.51" y="40.005" size="1.778" layer="27" font="vector" ratio="10" rot="R180" display="off"/>
 <attribute name="AMP" value="520151-4" x="16.51" y="40.005" size="1.778" layer="27" font="vector" ratio="10" rot="R180" display="off"/>
