File: Adapter-RJ45-SignalHead_array.brd (EAGLE design)
At the start: 119.4 x 110.5 mm, 49 parts

Commit message: added values for connectors
Parts:
- CON1X11, CON1X12, CON1X21, CON1X22, CON2X11, CON2X12, CON2X21, CON2X22: value (none) -> 2mm
- CON3X11, CON3X12, CON3X21, CON3X22, CON4X11, CON4X12, CON4X21, CON4X22: value (none) -> 0.100
- J1X11, J1X12, J1X21, J1X22: value (none) -> RJ12/6
- R1X11, R1X12, R1X21, R1X22, R2X11, R2X12, R2X21, R2X22, R3X11, R3X12, R3X21, R3X22, R4X11, R4X12, R4X21, R4X22, R5X11, R5X12, R5X21, R5X22, R6X11, R6X12, R6X21, R6X22: value (none) -> 0R
- U$1X1: value (none) -> 10x10
Changed lines of the file:
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@@
 </autorouter>
 <elements>
-<element name="CON1X11" library="SPCoast" package="4P-2.0" value="" x="42.545" y="9.525"/>
-<element name="CON2X11" library="SPCoast" package="4P-2.0" value="" x="22.86" y="9.525"/>
-<element name="CON3X11" library="SPCoast" package="1X04_LOCK" value="" x="19.05" y="6.985"/>
-<element name="CON4X11" library="SPCoast" package="1X04_LOCK" value="" x="38.1" y="6.985"/>
-<element name="J1X11" library="SPCoast" package="RJ45-NO-SHIELD" value="" x="33.02" y="40.005" rot="R180"/>
-<element name="R1X11" library="SPCoast" package="CUT-R" value="" x="27.94" y="20.32" rot="R90"/>
-<element name="R2X11" library="SPCoast" package="CUT-R" value="" x="24.13" y="20.32" rot="R90"/>
-<element name="R3X11" library="SPCoast" package="CUT-R" value="" x="20.32" y="20.32" rot="R90"/>
-<element name="R4X11" library="SPCoast" package="CUT-R" value="" x="43.18" y="20.32" rot="R90"/>
-<element name="R5X11" library="SPCoast" package="CUT-R" value="" x="39.37" y="20.32" rot="R90"/>
-<element name="R6X11" library="SPCoast" package="CUT-R" value="" x="35.56" y="20.32" rot="R90"/>
+<element name="CON1X11" library="SPCoast" package="4P-2.0" value="2mm" x="42.545" y="9.525"/>
+<element name="CON2X11" library="SPCoast" package="4P-2.0" value="2mm" x="22.86" y="9.525"/>
+<element name="CON3X11" library="SPCoast" package="1X04_LOCK" value="0.100" x="19.05" y="6.985"/>
+<element name="CON4X11" library="SPCoast" package="1X04_LOCK" value="0.100" x="38.1" y="6.985"/>
+<element name="J1X11" library="SPCoast" package="RJ45-NO-SHIELD" value="RJ12/6" x="33.02" y="40.005" rot="R180"/>
+<element name="R1X11" library="SPCoast" package="CUT-R" value="0R" x="27.94" y="20.32" rot="R90"/>
+<element name="R2X11" library="SPCoast" package="CUT-R" value="0R" x="24.13" y="20.32" rot="R90"/>
+<element name="R3X11" library="SPCoast" package="CUT-R" value="0R" x="20.32" y="20.32" rot="R90"/>
+<element name="R4X11" library="SPCoast" package="CUT-R" value="0R" x="43.18" y="20.32" rot="R90"/>
+<element name="R5X11" library="SPCoast" package="CUT-R" value="0R" x="39.37" y="20.32" rot="R90"/>
+<element name="R6X11" library="SPCoast" package="CUT-R" value="0R" x="35.56" y="20.32" rot="R90"/>
 <element name="U$1X11" library="SPCoast" package="OSHW-LOGO-M" value="DOC-OSHW-LOGO-M" x="33.02" y="41.91"/>
-<element name="CON1X12" library="SPCoast" package="4P-2.0" value="" x="42.545" y="55.245"/>
-<element name="CON2X12" library="SPCoast" package="4P-2.0" value="" x="22.86" y="55.245"/>
-<element name="CON3X12" library="SPCoast" package="1X04_LOCK" value="" x="19.05" y="52.705"/>
-<element name="CON4X12" library="SPCoast" package="1X04_LOCK" value="" x="38.1" y="52.705"/>
-<element name="J1X12" library="SPCoast" package="RJ45-NO-SHIELD" value="" x="33.02" y="85.725" rot="R180"/>
-<element name="R1X12" library="SPCoast" package="CUT-R" value="" x="27.94" y="66.04" rot="R90"/>
-<element name="R2X12" library="SPCoast" package="CUT-R" value="" x="24.13" y="66.04" rot="R90"/>
-<element name="R3X12" library="SPCoast" package="CUT-R" value="" x="20.32" y="66.04" rot="R90"/>
-<element name="R4X12" library="SPCoast" package="CUT-R" value="" x="43.18" y="66.04" rot="R90"/>
-<element name="R5X12" library="SPCoast" package="CUT-R" value="" x="39.37" y="66.04" rot="R90"/>
-<element name="R6X12" library="SPCoast" package="CUT-R" value="" x="35.56" y="66.04" rot="R90"/>
+<element name="CON1X12" library="SPCoast" package="4P-2.0" value="2mm" x="42.545" y="55.245"/>
+<element name="CON2X12" library="SPCoast" package="4P-2.0" value="2mm" x="22.86" y="55.245"/>
+<element name="CON3X12" library="SPCoast" package="1X04_LOCK" value="0.100" x="19.05" y="52.705"/>
+<element name="CON4X12" library="SPCoast" package="1X04_LOCK" value="0.100" x="38.1" y="52.705"/>
+<element name="J1X12" library="SPCoast" package="RJ45-NO-SHIELD" value="RJ12/6" x="33.02" y="85.725" rot="R180"/>
+<element name="R1X12" library="SPCoast" package="CUT-R" value="0R" x="27.94" y="66.04" rot="R90"/>
+<element name="R2X12" library="SPCoast" package="CUT-R" value="0R" x="24.13" y="66.04" rot="R90"/>
+<element name="R3X12" library="SPCoast" package="CUT-R" value="0R" x="20.32" y="66.04" rot="R90"/>
+<element name="R4X12" library="SPCoast" package="CUT-R" value="0R" x="43.18" y="66.04" rot="R90"/>
+<element name="R5X12" library="SPCoast" package="CUT-R" value="0R" x="39.37" y="66.04" rot="R90"/>
+<element name="R6X12" library="SPCoast" package="CUT-R" value="0R" x="35.56" y="66.04" rot="R90"/>
 <element name="U$1X12" library="SPCoast" package="OSHW-LOGO-M" value="DOC-OSHW-LOGO-M" x="33.02" y="87.63"/>
-<element name="CON1X21" library="SPCoast" package="4P-2.0" value="" x="75.565" y="9.525"/>
-<element name="CON2X21" library="SPCoast" package="4P-2.0" value="" x="55.88" y="9.525"/>
-<element name="CON3X21" library="SPCoast" package="1X04_LOCK" value="" x="52.07" y="6.985"/>
-<element name="CON4X21" library="SPCoast" package="1X04_LOCK" value="" x="71.12" y="6.985"/>
-<element name="J1X21" library="SPCoast" package="RJ45-NO-SHIELD" value="" x="66.04" y="40.005" rot="R180"/>
-<element name="R1X21" library="SPCoast" package="CUT-R" value="" x="60.96" y="20.32" rot="R90"/>
-<element name="R2X21" library="SPCoast" package="CUT-R" value="" x="57.15" y="20.32" rot="R90"/>
-<element name="R3X21" library="SPCoast" package="CUT-R" value="" x="53.34" y="20.32" rot="R90"/>
-<element name="R4X21" library="SPCoast" package="CUT-R" value="" x="76.2" y="20.32" rot="R90"/>
-<element name="R5X21" library="SPCoast" package="CUT-R" value="" x="72.39" y="20.32" rot="R90"/>
-<element name="R6X21" library="SPCoast" package="CUT-R" value="" x="68.58" y="20.32" rot="R90"/>
+<element name="CON1X21" library="SPCoast" package="4P-2.0" value="2mm" x="75.565" y="9.525"/>
+<element name="CON2X21" library="SPCoast" package="4P-2.0" value="2mm" x="55.88" y="9.525"/>
+<element name="CON3X21" library="SPCoast" package="1X04_LOCK" value="0.100" x="52.07" y="6.985"/>
+<element name="CON4X21" library="SPCoast" package="1X04_LOCK" value="0.100" x="71.12" y="6.985"/>
+<element name="J1X21" library="SPCoast" package="RJ45-NO-SHIELD" value="RJ12/6" x="66.04" y="40.005" rot="R180"/>
+<element name="R1X21" library="SPCoast" package="CUT-R" value="0R" x="60.96" y="20.32" rot="R90"/>
+<element name="R2X21" library="SPCoast" package="CUT-R" value="0R" x="57.15" y="20.32" rot="R90"/>
+<element name="R3X21" library="SPCoast" package="CUT-R" value="0R" x="53.34" y="20.32" rot="R90"/>
+<element name="R4X21" library="SPCoast" package="CUT-R" value="0R" x="76.2" y="20.32" rot="R90"/>
+<element name="R5X21" library="SPCoast" package="CUT-R" value="0R" x="72.39" y="20.32" rot="R90"/>
+<element name="R6X21" library="SPCoast" package="CUT-R" value="0R" x="68.58" y="20.32" rot="R90"/>
 <element name="U$1X21" library="SPCoast" package="OSHW-LOGO-M" value="DOC-OSHW-LOGO-M" x="66.04" y="41.91"/>
-<element name="CON1X22" library="SPCoast" package="4P-2.0" value="" x="75.565" y="55.245"/>
-<element name="CON2X22" library="SPCoast" package="4P-2.0" value="" x="55.88" y="55.245"/>
-<element name="CON3X22" library="SPCoast" package="1X04_LOCK" value="" x="52.07" y="52.705"/>
-<element name="CON4X22" library="SPCoast" package="1X04_LOCK" value="" x="71.12" y="52.705"/>
-<element name="J1X22" library="SPCoast" package="RJ45-NO-SHIELD" value="" x="66.04" y="85.725" rot="R180"/>
-<element name="R1X22" library="SPCoast" package="CUT-R" value="" x="60.96" y="66.04" rot="R90"/>
-<element name="R2X22" library="SPCoast" package="CUT-R" value="" x="57.15" y="66.04" rot="R90"/>
-<element name="R3X22" library="SPCoast" package="CUT-R" value="" x="53.34" y="66.04" rot="R90"/>
-<element name="R4X22" library="SPCoast" package="CUT-R" value="" x="76.2" y="66.04" rot="R90"/>
-<element name="R5X22" library="SPCoast" package="CUT-R" value="" x="72.39" y="66.04" rot="R90"/>
-<element name="R6X22" library="SPCoast" package="CUT-R" value="" x="68.58" y="66.04" rot="R90"/>
+<element name="CON1X22" library="SPCoast" package="4P-2.0" value="2mm" x="75.565" y="55.245"/>
+<element name="CON2X22" library="SPCoast" package="4P-2.0" value="2mm" x="55.88" y="55.245"/>
+<element name="CON3X22" library="SPCoast" package="1X04_LOCK" value="0.100" x="52.07" y="52.705"/>
+<element name="CON4X22" library="SPCoast" package="1X04_LOCK" value="0.100" x="71.12" y="52.705"/>
+<element name="J1X22" library="SPCoast" package="RJ45-NO-SHIELD" value="RJ12/6" x="66.04" y="85.725" rot="R180"/>
+<element name="R1X22" library="SPCoast" package="CUT-R" value="0R" x="60.96" y="66.04" rot="R90"/>
+<element name="R2X22" library="SPCoast" package="CUT-R" value="0R" x="57.15" y="66.04" rot="R90"/>
+<element name="R3X22" library="SPCoast" package="CUT-R" value="0R" x="53.34" y="66.04" rot="R90"/>
+<element name="R4X22" library="SPCoast" package="CUT-R" value="0R" x="76.2" y="66.04" rot="R90"/>
+<element name="R5X22" library="SPCoast" package="CUT-R" value="0R" x="72.39" y="66.04" rot="R90"/>
+<element name="R6X22" library="SPCoast" package="CUT-R" value="0R" x="68.58" y="66.04" rot="R90"/>
 <element name="U$1X22" library="SPCoast" package="OSHW-LOGO-M" value="DOC-OSHW-LOGO-M" x="66.04" y="87.63"/>
-<element name="U$1X1" library="SPCoast" package="BOARD-SEEED10X10-NOHOLES" value="" x="0" y="0"/>
+<element name="U$1X1" library="SPCoast" package="BOARD-SEEED10X10-NOHOLES" value="10x10" x="0" y="0"/>
 </elements>
 <signals>

Commit message: normalized values
Parts:
- J1X11, J1X12, J1X21, J1X22: value RJ12/6 -> RJ45
- R1X11, R1X12, R1X21, R1X22, R2X11, R2X12, R2X21, R2X22, R3X11, R3X12, R3X21, R3X22, R4X11, R4X12, R4X21, R4X22, R5X11, R5X12, R5X21, R5X22, R6X11, R6X12, R6X21, R6X22: value 0R -> nostuff
- U$1X1: value 10x10 -> BOARD
- U$1X11, U$1X12, U$1X21, U$1X22: value DOC-OSHW-LOGO-M -> OSHW
Changed lines of the file:
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@@
 <element name="CON3X11" library="SPCoast" package="1X04_LOCK" value="0.100" x="19.05" y="6.985"/>
 <element name="CON4X11" library="SPCoast" package="1X04_LOCK" value="0.100" x="38.1" y="6.985"/>
-<element name="J1X11" library="SPCoast" package="RJ45-NO-SHIELD" value="RJ12/6" x="33.02" y="40.005" rot="R180"/>
-<element name="R1X11" library="SPCoast" package="CUT-R" value="0R" x="27.94" y="20.32" rot="R90"/>
-<element name="R2X11" library="SPCoast" package="CUT-R" value="0R" x="24.13" y="20.32" rot="R90"/>
-<element name="R3X11" library="SPCoast" package="CUT-R" value="0R" x="20.32" y="20.32" rot="R90"/>
-<element name="R4X11" library="SPCoast" package="CUT-R" value="0R" x="43.18" y="20.32" rot="R90"/>
-<element name="R5X11" library="SPCoast" package="CUT-R" value="0R" x="39.37" y="20.32" rot="R90"/>
-<element name="R6X11" library="SPCoast" package="CUT-R" value="0R" x="35.56" y="20.32" rot="R90"/>
-<element name="U$1X11" library="SPCoast" package="OSHW-LOGO-M" value="DOC-OSHW-LOGO-M" x="33.02" y="41.91"/>
+<element name="J1X11" library="SPCoast" package="RJ45-NO-SHIELD" value="RJ45" x="33.02" y="40.005" rot="R180"/>
+<element name="R1X11" library="SPCoast" package="CUT-R" value="nostuff" x="27.94" y="20.32" rot="R90"/>
+<element name="R2X11" library="SPCoast" package="CUT-R" value="nostuff" x="24.13" y="20.32" rot="R90"/>
+<element name="R3X11" library="SPCoast" package="CUT-R" value="nostuff" x="20.32" y="20.32" rot="R90"/>
+<element name="R4X11" library="SPCoast" package="CUT-R" value="nostuff" x="43.18" y="20.32" rot="R90"/>
+<element name="R5X11" library="SPCoast" package="CUT-R" value="nostuff" x="39.37" y="20.32" rot="R90"/>
+<element name="R6X11" library="SPCoast" package="CUT-R" value="nostuff" x="35.56" y="20.32" rot="R90"/>
+<element name="U$1X11" library="SPCoast" package="OSHW-LOGO-M" value="OSHW" x="33.02" y="41.91"/>
 <element name="CON1X12" library="SPCoast" package="4P-2.0" value="2mm" x="42.545" y="55.245"/>
 <element name="CON2X12" library="SPCoast" package="4P-2.0" value="2mm" x="22.86" y="55.245"/>
 <element name="CON3X12" library="SPCoast" package="1X04_LOCK" value="0.100" x="19.05" y="52.705"/>
 <element name="CON4X12" library="SPCoast" package="1X04_LOCK" value="0.100" x="38.1" y="52.705"/>
-<element name="J1X12" library="SPCoast" package="RJ45-NO-SHIELD" value="RJ12/6" x="33.02" y="85.725" rot="R180"/>
-<element name="R1X12" library="SPCoast" package="CUT-R" value="0R" x="27.94" y="66.04" rot="R90"/>
-<element name="R2X12" library="SPCoast" package="CUT-R" value="0R" x="24.13" y="66.04" rot="R90"/>
-<element name="R3X12" library="SPCoast" package="CUT-R" value="0R" x="20.32" y="66.04" rot="R90"/>
-<element name="R4X12" library="SPCoast" package="CUT-R" value="0R" x="43.18" y="66.04" rot="R90"/>
-<element name="R5X12" library="SPCoast" package="CUT-R" value="0R" x="39.37" y="66.04" rot="R90"/>
-<element name="R6X12" library="SPCoast" package="CUT-R" value="0R" x="35.56" y="66.04" rot="R90"/>
-<element name="U$1X12" library="SPCoast" package="OSHW-LOGO-M" value="DOC-OSHW-LOGO-M" x="33.02" y="87.63"/>
+<element name="J1X12" library="SPCoast" package="RJ45-NO-SHIELD" value="RJ45" x="33.02" y="85.725" rot="R180"/>
+<element name="R1X12" library="SPCoast" package="CUT-R" value="nostuff" x="27.94" y="66.04" rot="R90"/>
+<element name="R2X12" library="SPCoast" package="CUT-R" value="nostuff" x="24.13" y="66.04" rot="R90"/>
+<element name="R3X12" library="SPCoast" package="CUT-R" value="nostuff" x="20.32" y="66.04" rot="R90"/>
+<element name="R4X12" library="SPCoast" package="CUT-R" value="nostuff" x="43.18" y="66.04" rot="R90"/>
+<element name="R5X12" library="SPCoast" package="CUT-R" value="nostuff" x="39.37" y="66.04" rot="R90"/>
+<element name="R6X12" library="SPCoast" package="CUT-R" value="nostuff" x="35.56" y="66.04" rot="R90"/>
+<element name="U$1X12" library="SPCoast" package="OSHW-LOGO-M" value="OSHW" x="33.02" y="87.63"/>
 <element name="CON1X21" library="SPCoast" package="4P-2.0" value="2mm" x="75.565" y="9.525"/>
 <element name="CON2X21" library="SPCoast" package="4P-2.0" value="2mm" x="55.88" y="9.525"/>
 <element name="CON3X21" library="SPCoast" package="1X04_LOCK" value="0.100" x="52.07" y="6.985"/>
 <element name="CON4X21" library="SPCoast" package="1X04_LOCK" value="0.100" x="71.12" y="6.985"/>
-<element name="J1X21" library="SPCoast" package="RJ45-NO-SHIELD" value="RJ12/6" x="66.04" y="40.005" rot="R180"/>
-<element name="R1X21" library="SPCoast" package="CUT-R" value="0R" x="60.96" y="20.32" rot="R90"/>
-<element name="R2X21" library="SPCoast" package="CUT-R" value="0R" x="57.15" y="20.32" rot="R90"/>
-<element name="R3X21" library="SPCoast" package="CUT-R" value="0R" x="53.34" y="20.32" rot="R90"/>
-<element name="R4X21" library="SPCoast" package="CUT-R" value="0R" x="76.2" y="20.32" rot="R90"/>
-<element name="R5X21" library="SPCoast" package="CUT-R" value="0R" x="72.39" y="20.32" rot="R90"/>
-<element name="R6X21" library="SPCoast" package="CUT-R" value="0R" x="68.58" y="20.32" rot="R90"/>
-<element name="U$1X21" library="SPCoast" package="OSHW-LOGO-M" value="DOC-OSHW-LOGO-M" x="66.04" y="41.91"/>
+<element name="J1X21" library="SPCoast" package="RJ45-NO-SHIELD" value="RJ45" x="66.04" y="40.005" rot="R180"/>
+<element name="R1X21" library="SPCoast" package="CUT-R" value="nostuff" x="60.96" y="20.32" rot="R90"/>
+<element name="R2X21" library="SPCoast" package="CUT-R" value="nostuff" x="57.15" y="20.32" rot="R90"/>
+<element name="R3X21" library="SPCoast" package="CUT-R" value="nostuff" x="53.34" y="20.32" rot="R90"/>
+<element name="R4X21" library="SPCoast" package="CUT-R" value="nostuff" x="76.2" y="20.32" rot="R90"/>
+<element name="R5X21" library="SPCoast" package="CUT-R" value="nostuff" x="72.39" y="20.32" rot="R90"/>
+<element name="R6X21" library="SPCoast" package="CUT-R" value="nostuff" x="68.58" y="20.32" rot="R90"/>
+<element name="U$1X21" library="SPCoast" package="OSHW-LOGO-M" value="OSHW" x="66.04" y="41.91"/>
 <element name="CON1X22" library="SPCoast" package="4P-2.0" value="2mm" x="75.565" y="55.245"/>
 <element name="CON2X22" library="SPCoast" package="4P-2.0" value="2mm" x="55.88" y="55.245"/>
 <element name="CON3X22" library="SPCoast" package="1X04_LOCK" value="0.100" x="52.07" y="52.705"/>
 <element name="CON4X22" library="SPCoast" package="1X04_LOCK" value="0.100" x="71.12" y="52.705"/>
-<element name="J1X22" library="SPCoast" package="RJ45-NO-SHIELD" value="RJ12/6" x="66.04" y="85.725" rot="R180"/>
-<element name="R1X22" library="SPCoast" package="CUT-R" value="0R" x="60.96" y="66.04" rot="R90"/>
-<element name="R2X22" library="SPCoast" package="CUT-R" value="0R" x="57.15" y="66.04" rot="R90"/>
-<element name="R3X22" library="SPCoast" package="CUT-R" value="0R" x="53.34" y="66.04" rot="R90"/>
-<element name="R4X22" library="SPCoast" package="CUT-R" value="0R" x="76.2" y="66.04" rot="R90"/>
-<element name="R5X22" library="SPCoast" package="CUT-R" value="0R" x="72.39" y="66.04" rot="R90"/>
-<element name="R6X22" library="SPCoast" package="CUT-R" value="0R" x="68.58" y="66.04" rot="R90"/>
-<element name="U$1X22" library="SPCoast" package="OSHW-LOGO-M" value="DOC-OSHW-LOGO-M" x="66.04" y="87.63"/>
-<element name="U$1X1" library="SPCoast" package="BOARD-SEEED10X10-NOHOLES" value="10x10" x="0" y="0"/>
+<element name="J1X22" library="SPCoast" package="RJ45-NO-SHIELD" value="RJ45" x="66.04" y="85.725" rot="R180"/>
+<element name="R1X22" library="SPCoast" package="CUT-R" value="nostuff" x="60.96" y="66.04" rot="R90"/>
+<element name="R2X22" library="SPCoast" package="CUT-R" value="nostuff" x="57.15" y="66.04" rot="R90"/>
+<element name="R3X22" library="SPCoast" package="CUT-R" value="nostuff" x="53.34" y="66.04" rot="R90"/>
+<element name="R4X22" library="SPCoast" package="CUT-R" value="nostuff" x="76.2" y="66.04" rot="R90"/>
+<element name="R5X22" library="SPCoast" package="CUT-R" value="nostuff" x="72.39" y="66.04" rot="R90"/>
+<element name="R6X22" library="SPCoast" package="CUT-R" value="nostuff" x="68.58" y="66.04" rot="R90"/>
+<element name="U$1X22" library="SPCoast" package="OSHW-LOGO-M" value="OSHW" x="66.04" y="87.63"/>
+<element name="U$1X1" library="SPCoast" package="BOARD-SEEED10X10-NOHOLES" value="BOARD" x="0" y="0"/>
 </elements>
 <signals>
